Commit message: Update car.urdf

File: src/my_car/urdf/car.urdf (robot description, URDF)
Before this commit: robot diff_car, 4 links, 3 joints
Links:
- link base_link: mass None -> 1.0
- link caster_wheel: mass None -> 0.05; geometry collision sphere radius=0.03; visual sphere radius=0.03
- link left_wheel: mass None -> 0.1; geometry collision cylinder length=0.04 radius=0.05; visual cylinder length=0.04 radius=0.05
- link right_wheel: mass None -> 0.1; geometry collision cylinder length=0.04 radius=0.05; visual cylinder length=0.04 radius=0.05
Joints:
- removed joint left_joint
- removed joint right_joint
- added joint left_wheel_joint: type continuous, parent base_link, child left_wheel, origin xyz=0 -0.1 0.05 rpy=0 0 0, axis 0 1 0, limit effort=1000 velocity=10
- added joint right_wheel_joint: type continuous, parent base_link, child right_wheel, origin xyz=0 0.1 0.05 rpy=0 0 0, axis 0 1 0, limit effort=1000 velocity=10
- joint caster_joint: origin xyz=-0.15 0 -0.02 rpy=0 0 0 -> xyz=-0.15 0 0.03 rpy=0 0 0
