Commit message: fix(ground): 修正机器人生成后自转 90°、rviz 看不到激光的问题
在虚拟机里用 GUI 实跑时发现：机器人不受指令就会自己转到 -90° 并滑到墙边
（真值 (-3.5,0,0) → (-3.24,-0.70,-90°)），定位因此永远收敛不了；
同时 rviz 里只有粒子云，没有激光点。逐个查下来是四个问题：

1. 车体碰撞盒底部正好在 z=0，与地面刮擦。
   碰撞盒中心从 0.08 抬到 0.10（底部留 2 cm 间隙），视觉与碰撞盒同步。

2. 轮子碰撞体用圆柱 —— 圆柱侧面与地面是**线接触**，接触求解容易产生
   粘滑振荡，表现为"机器人自己打转"。碰撞体改成球体（半径 0.1），
   圆柱只保留为外观。改完后静止 8 秒位移 0.0000 m、航向变化 0.00°。

3. 世界刚启动就 spawn 模型。gazebo 前几秒物理还没稳定，
   立刻生成会被接触求解推走，而且每次都被推到同一个（错误的）位姿——
   看起来完全像"定位算法不收敛"，极难排查。
   spawn 加 5 秒延迟（launch-prefix 里 sleep，参数 spawn_delay 可调）后，
   机器人精确停在 (-3.500, 0.000, 0.00°)。

4. 没有 robot_state_publisher，URDF 里的固定关节（base_link -> laser_link）
   不产生 TF，rviz 无法把激光变换到 map 系。
   加入 robot_state_publisher，并把原来的静态 TF 去掉（避免与它冲突）。
   现在 TF 链完整：map -> odom -> base_footprint -> base_link -> laser_link。

验证（Ubuntu 20.04 + Noetic + Gazebo 11，无头）：
- 静止 8 秒：位移 0.0000 m，航向变化 0.00°；
- MCL 起点误差 0.071 m / 0.1°；直行 4 s 后 0.066 m / 0.2°；
  转向再直行后 0.050 m / 7.6°（同期里程计累计漂移 0.284 m）；
- TF map->laser_link 存在。

File: src/ground/lidar_mcl_localization/urdf/mcl_bot.urdf (robot description, URDF)
Before this commit: robot mcl_bot, 7 links, 6 joints
Links:
- link wheel_l: geometry collision sphere radius=0.100; visual cylinder length=0.040 radius=0.100
- link wheel_r: geometry collision sphere radius=0.100; visual cylinder length=0.040 radius=0.100
